File: hardware/buuc.kicad_pcb (KiCad board)
At the start: 2 copper layers, 15 parts, among them P1 USB_OTG, P2 CONN_01X02, Q1 NDS8434, U1 BOOST_REGULATOR, U2 MCP73842-840I/UN

Commit message: Minor pcb changes.
Other:
- board outline added: 45.1 x 29.8 mm
- net class Default: trace_width 0.5 -> 0.25
Changed lines of the file:
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@@
-(kicad_pcb (version 20160815) (host pcbnew "(2016-12-18 revision 3ffa37c)-master")
+(kicad_pcb (version 20170123) (host pcbnew no-vcs-found-1fe91e6~59~ubuntu16.04.1)
   (general
-    (links 33)
-    (no_connects 0)
-    (area 136.525 50.46961 181.9725 81.9325)
     (thickness 1.6)
-    (drawings 0)
+    (drawings 4)
     (tracks 96)
     (zones 0)
@@
     (nets 17)
   )
-  (page A4)
+  (page USLetter)
   (layers
     (0 F.Cu signal)
@@
   )
   (setup
-    (last_trace_width 0.5)
+    (last_trace_width 0.25)
     (user_trace_width 0.25)
     (user_trace_width 0.35)
@@
     (visible_elements FFFFFF7F)
     (pcbplotparams
-      (layerselection 0x00030_ffffffff)
+      (layerselection 0x000c0_ffffffff)
       (usegerberextensions false)
+      (usegerberattributes true)
+      (usegerberadvancedattributes true)
+      (creategerberjobfile true)
       (excludeedgelayer true)
       (linewidth 0.100000)
       (plotframeref false)
-      (viasonmask false)
+      (viasonmask true)
       (mode 1)
-      (useauxorigin false)
+      (useauxorigin true)
       (hpglpennumber 1)
       (hpglpenspeed 20)
@@
       (outputformat 1)
       (mirror false)
-      (drillshape 1)
+      (drillshape 0)
       (scaleselection 1)
       (outputdirectory ""))
@@
   (net_class Default "This is the default net class."
     (clearance 0.2)
-    (trace_width 0.5)
+    (trace_width 0.25)
     (via_dia 1.5)
     (via_drill 0.5)
     (uvia_dia 0.3)
     (uvia_drill 0.1)
-    (diff_pair_gap 0.25)
-    (diff_pair_width 0.2)
     (add_net +5V)
     (add_net +BATT)
@@
     )
   )
+  (gr_line (start 135.89 81.28) (end 135.89 51.435) (angle 90) (layer Edge.Cuts) (width 0.15))
+  (gr_line (start 180.975 81.28) (end 135.89 81.28) (angle 90) (layer Edge.Cuts) (width 0.15))
+  (gr_line (start 180.975 51.435) (end 180.975 81.28) (angle 90) (layer Edge.Cuts) (width 0.15))
+  (gr_line (start 135.89 51.435) (end 180.975 51.435) (angle 90) (layer Edge.Cuts) (width 0.15))
   (segment (start 164.125 65.905) (end 169.045 65.905) (width 0.25) (layer F.Cu) (net 1))
   (segment (start 169.045 65.905) (end 170.26 64.69) (width 0.25) (layer F.Cu) (net 1))
