File: hardware/buuc.sch (KiCad schematic (older format))
At the start: 17 parts, among them P1 USB_OTG, P2 CONN_01X02, Q1 NDS8434, U1 BOOST_REGULATOR, U2 MCP73842-840I/UN

Commit message: If I'm going to do this another time, I might as well make it count.
Parts:
- removed P2: CONN_01X02, myelin/myelin-kicad.pretty:header_01x02_40mil_60mil, symbol CONN_01X02
- added J1: RADIO+, coddingtonbear/coddingtonbear.pretty:TAB, symbol Conn_01x01
- added J2: RADIO-, coddingtonbear/coddingtonbear.pretty:TAB, symbol Conn_01x01
- C1, C2: value 10u -> 22uF; footprint pelrun/libKiCad/footprint/w_smd_cap.pretty:c_elec_5x5.8 -> KiCad/Capacitors_SMD.pretty:C_1206_HandSoldering
- P1: footprint coddingtonbear/coddingtonbear.pretty:USB_Thru_hole -> coddingtonbear/coddingtonbear.pretty:UJ2-MIBH-4-SMT
Connections:
- net +BATT: now also J1.1 (Pin_1)
- net GND: now also P1.6 (shield), J2.1 (Pin_1)
Changed lines of the file:
@@
-EESchema Schematic File Version 2
+EESchema Schematic File Version 3
 LIBS:buuc-rescue
 LIBS:power
@@
 F 0 "P1" V 1580 1638 50  0000 L CNN
 F 1 "USB_OTG" V 1671 1638 50  0000 L CNN
-F 2 "coddingtonbear/coddingtonbear.pretty:USB_Thru_hole" V 1500 1350 50  0001 C CNN
+F 2 "coddingtonbear/coddingtonbear.pretty:UJ2-MIBH-4-SMT" V 1500 1350 50  0001 C CNN
 F 3 "" V 1500 1350 50  0000 C CNN
 	1    1550 1450
@@
 P 3100 3250
 F 0 "C1" H 3218 3296 50  0000 L CNN
-F 1 "10u" H 3218 3205 50  0000 L CNN
-F 2 "pelrun/libKiCad/footprint/w_smd_cap.pretty:c_elec_5x5.8" H 3138 3100 50  0001 C CNN
+F 1 "22uF" H 3218 3205 50  0000 L CNN
+F 2 "KiCad/Capacitors_SMD.pretty:C_1206_HandSoldering" H 3138 3100 50  0001 C CNN
 F 3 "" H 3100 3250 50  0000 C CNN
 	1    3100 3250
@@
 P 5650 3550
 F 0 "C2" H 5768 3596 50  0000 L CNN
-F 1 "10u" H 5768 3505 50  0000 L CNN
-F 2 "pelrun/libKiCad/footprint/w_smd_cap.pretty:c_elec_5x5.8" H 5688 3400 50  0001 C CNN
+F 1 "22uF" H 5768 3505 50  0000 L CNN
+F 2 "KiCad/Capacitors_SMD.pretty:C_1206_HandSoldering" H 5688 3400 50  0001 C CNN
 F 3 "" H 5650 3550 50  0000 C CNN
 	1    5650 3550
@@
 Text Notes 2400 2550 0    60   ~ 0
 VCC: 8.7V-12V
-$Comp
-L CONN_01X02 P2
-U 1 1 59AF80AC
-P 6550 2700
-F 0 "P2" H 6628 2741 50  0000 L CNN
-F 1 "CONN_01X02" H 6628 2650 50  0000 L CNN
-F 2 "myelin/myelin-kicad.pretty:header_01x02_40mil_60mil" H 6550 2700 50  0001 C CNN
-F 3 "" H 6550 2700 50  0000 C CNN
-	1    6550 2700
-	1    0    0    -1
-$EndComp
 $Comp
 L R R3
@@
 Wire Wire Line
 	1850 1650 2000 1650
+$Comp
+L Conn_01x01 J1
+U 1 1 59D1854E
+P 6550 2650
+F 0 "J1" H 6630 2692 50  0000 L CNN
+F 1 "RADIO+" H 6630 2601 50  0000 L CNN
+F 2 "coddingtonbear/coddingtonbear.pretty:TAB" H 6550 2650 50  0001 C CNN
+F 3 "" H 6550 2650 50  0001 C CNN
+	1    6550 2650
+	1    0    0    -1
+$EndComp
+$Comp
+L Conn_01x01 J2
+U 1 1 59D18593
+P 6550 2750
+F 0 "J2" H 6630 2792 50  0000 L CNN
+F 1 "RADIO-" H 6630 2701 50  0000 L CNN
+F 2 "coddingtonbear/coddingtonbear.pretty:TAB" H 6550 2750 50  0001 C CNN
+F 3 "" H 6550 2750 50  0001 C CNN
+	1    6550 2750
+	1    0    0    -1
+$EndComp
+Wire Wire Line
+	1900 1250 1900 1050
+Wire Wire Line
+	1900 1050 1450 1050
+Connection ~ 1900 1250
 $EndSCHEMATC
